File: docs/kicad_project/ea801_cvt/ea801_cvt.kicad_sch (KiCad schematic)
At the start: 8 parts, among them J2_BitDogLab Conn_01x06_MountingPin, J2_BitDogLab1 J2_IDC_BitDogLab, M1 Motor principal, M2 Motor Fuso Câmbio, U1 L293D

Commit message: att kicad project
Parts:
- removed D1, D2: 1N4007, Diode_THT:D_DO-41_SOD81_P10.16mm_Horizontal, symbol Diode:1N4007
